File: 3V3.kicad_sch (KiCad schematic)
At the start: 16 parts, among them U2 A6986F

Commit message: Buck-boost 5V entry
Parts:
- renumbered C6 to C11, C1 to C13, C4 to C15, C3 to C16, C7 to C17, C5 to C18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
Connections:
- net BUS3V3 renamed BUS5V
