File: HEDGE-Comm/LTC3225fb.kicad_sch (KiCad schematic)
At the start: 9 parts, among them U1 LTC3225EDDB-TRMPBF

Commit message: Refactor Data PCB files; enter RS485; enter Iridium radio power
Other:
- title: HEDGE-Data PCB -> HEDGE Comm PCB
Changed lines of the file:
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@@
 	(paper "C")
 	(title_block
-		(title "HEDGE-Data PCB")
-		(date "2024-10-09")
+		(title "HEDGE Comm PCB")
+		(date "2024-10-11")
 		(rev "1.0")
 		(company "Spacecraft Design Lab")
